Commit message: Turn off green starbucks bottle collisions and remove velocity obs and fix blue robot vis

File: source/isaaclab_assets/data/kiri/green_starbucks_bottle/urdf/starbucks_bottle.urdf (robot description, URDF)
Before this commit: robot model.urdf, 1 links, 0 joints
Links:
- link baseLink: geometry visual mesh filename=starbucks_bottle.obj scale=1 1 1
